File: hw/lpc1549.sch (KiCad schematic (older format))
At the start: 15 parts, among them J301 ARM_JTAG_SWD_HEADER_10_PINSMD, U301 MCP2551_SOIC8, U302 LPC1549JBD64, X301 XTAL_7A-12.000MAAJ-T

Commit message: 1.0 pcb created
Parts:
- removed J301: ARM_JTAG_SWD_HEADER_10_PINSMD, usevolt:ARM_10_PIN_JTAG_SWD_CONNECTOR, symbol ARM_JTAG_SWD_HEADER_10_PINSMD
- added J201: ARM_JTAG_SWD_HEADER_10_PINSMD, usevolt:ARM_10_PIN_JTAG_SWD_CONNECTOR, symbol usevolt:ARM_JTAG_SWD_HEADER_10_PINSMD
- C201: renamed from C301; symbol 100nF -> kemet:100nF
- C202: renamed from C302; symbol 100nF -> kemet:100nF
- C203: renamed from C303; symbol 100nF -> kemet:100nF
- C204: renamed from C304; symbol 100nF -> kemet:100nF
- C205: renamed from C305; symbol 100nF -> kemet:100nF
- C206: renamed from C306; symbol 100nF -> kemet:100nF
- C207: renamed from C307; symbol 100nF -> kemet:100nF
- C208: renamed from C308; symbol 18pF -> kemet:18pF
- C209: renamed from C309; symbol 18pF -> kemet:18pF
- R201: renamed from R301; symbol 10K -> yageo:10K
- R202: renamed from R302; symbol 10K -> yageo:10K
- U201: renamed from U301; symbol MCP2551_SOIC8 -> usevolt:MCP2551_SOIC8
- U202: renamed from U302; symbol LPC1549JBD64 -> usevolt:LPC1549JBD64
- X201: renamed from X301; symbol XTAL_7A-12.000MAAJ-T -> usevolt:XTAL_7A-12.000MAAJ-T
Connections:
- net labels added: OUT10_1, OUT10_2, OUT10_SENSE, OUT11, OUT11_SENSE, OUT1_1, OUT1_2, OUT1_SENSE, OUT2_1, OUT2_2, OUT2_SENSE, OUT3_1, OUT3_2, OUT3_SENSE, OUT4_1, OUT4_2, OUT4_SENSE, OUT5_1, OUT5_2, OUT5_SENSE, OUT6_1, OUT6_2, OUT6_SENSE, OUT7_1, OUT7_2, OUT7_SENSE, OUT8_1, OUT8_2, OUT8_SENSE, OUT9_1, OUT9_2, OUT9_SENSE, PRESS_SENSE
- net labels removed: AC, AC_SENSE, ALT_IG, ALT_IG_SENSE, ALT_L, ALT_P/RPM, FUEL_LEVEL, GLOW_PLUGS, GLOW_PLUGS_SENSE, HYDR_OIL_TEMP, MOTOR_OIL_PRESS, MOTOR_ON, MOTOR_ON_SENSE, MOTOR_START, MOTOR_START_SENSE, MOTOR_TEMP, MOTOR_WATER_TEMP, OILC, OILC_SENSE, OIL_LEVEL, PUMP, PUMP_SENSE, STARTER, STARTER_SENSE, VDD_SENSE
- wire segments 80 -> 117
