File: hw/pwr_supply_sheet.sch (KiCad schematic (older format))
At the start: 17 parts

Commit message: 1.0 pcb created
Parts:
- removed D202, D205: SCHOTTKY_DIODE_V40PW10C, usevolt:SlimDPAK, symbol SCHOTTKY_DIODE_V40PW10C
- removed R201: 10K, multicomp:0603, symbol 10K
- removed R202: 1K, multicomp:0603, symbol 1K
- C1301: renamed from C201; symbol 100nF -> kemet:100nF
- C1302: renamed from C202; symbol CAP_EEE-FK1H470P -> usevolt:CAP_EEE-FK1H470P
- C1303: renamed from C203; symbol 10nF -> kemet:10nF
- C1304: renamed from C204; symbol T491D226K035AT -> kemet:T491D226K035AT
- C1305: renamed from C205; symbol 100nF -> kemet:100nF
- D1301: renamed from D201; symbol DIODE_RS07J-GS18 -> usevolt:DIODE_RS07J-GS18
- D1302: renamed from D203; symbol DIODE_TVS_SMBJ33A-TRDO-214AA -> usevolt:DIODE_TVS_SMBJ33A-TRDO-214AA
- D1303: renamed from D206; symbol DIODE_TVS_TPSMD28A -> usevolt:DIODE_TVS_TPSMD28A
- D1304: renamed from D204; symbol DIODE_RS07J-GS18 -> usevolt:DIODE_RS07J-GS18
- F1301: renamed from F201; symbol FUSE_MC36211_350MA -> usevolt:FUSE_MC36211_350MA
- L1301: renamed from L201; symbol IND_744045210 -> usevolt:IND_744045210
- VR1301: renamed from VR201; symbol LM2671SOIC8 -> usevolt:LM2671SOIC8
- VR1302: renamed from VR202; symbol REG_MCP1700 -> usevolt:REG_MCP1700
Connections:
- net labels removed: VDD_SENSE
- wire segments 40 -> 47
