File: hw/hcu.kicad_pcb (KiCad board)
At the start: 2 copper layers, 78 x 90 mm, 122 parts, among them J101 AMPSEAL_23_POS_VERT_BLACK_SEA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, J102 AMPSEAL_8_POS_VERT_WHITE_SEAL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, J201 ARM_JTAG_SWD_HEADER_10_PINSMD, U1001 VND5050AJTR-E, U1101 VND5050AJTR-E, U1201 VND5050AJTR-E, U1401 VN5E010AH, U201 MCP2551_SOIC8, U202 LPC1549JBD64, U301 VND5050AJTR-E, U401 VND5050AJTR-E, U501 VND5050AJTR-E, U601 VND5050AJTR-E, U701 VND5050AJTR-E, U801 VND5050AJTR-E, U901 VND5050AJTR-E, X201 XTAL_7A-12.000MAAJ-T

Commit message: pcb 1.3.0 created
Parts:
- added R1: 120, yageo:0603, B.Cu at (176.3, 122.9)
Connections:
- J102 pad 6: (no net) -> Net-(J102-Pad6)
- J102 pad 7: (no net) -> Net-(J102-Pad7)
- J102 pad 8: (no net) -> Net-(J102-Pad8)
- J201 pad P$6: (no net) -> Net-(J201-PadP$6)
- J201 pad P$7: (no net) -> Net-(J201-PadP$7)
- J201 pad P$8: (no net) -> Net-(J201-PadP$8)
- U1001 pad 6: (no net) -> Net-(U1001-Pad6)
- U1101 pad 6: (no net) -> Net-(U1101-Pad6)
- U1201 pad 6: (no net) -> Net-(U1201-Pad6)
- U201 pad 5: (no net) -> Net-(U201-Pad5)
- U202 pad P$24: (no net) -> Net-(U202-PadP$24)
- U202 pad P$38: (no net) -> Net-(U202-PadP$38)
- U202 pad P$39: (no net) -> Net-(U202-PadP$39)
- U202 pad P$42: (no net) -> Net-(U202-PadP$42)
- U202 pad P$43: (no net) -> Net-(U202-PadP$43)
- U202 pad P$47: (no net) -> Net-(U202-PadP$47)
- U202 pad P$48: (no net) -> Net-(U202-PadP$48)
- U202 pad P$49: (no net) -> Net-(U202-PadP$49)
- U202 pad P$50: (no net) -> Net-(U202-PadP$50)
- U202 pad P$54: (no net) -> Net-(U202-PadP$54)
- U301 pad 6: (no net) -> Net-(U301-Pad6)
- U401 pad 6: (no net) -> Net-(U401-Pad6)
- U501 pad 6: (no net) -> Net-(U501-Pad6)
- U601 pad 6: (no net) -> Net-(U601-Pad6)
- U701 pad 6: (no net) -> Net-(U701-Pad6)
- U801 pad 6: (no net) -> Net-(U801-Pad6)
- U901 pad 6: (no net) -> Net-(U901-Pad6)
- VR1301 pad 2: (no net) -> Net-(VR1301-Pad2)
- VR1301 pad 3: (no net) -> Net-(VR1301-Pad3)
- VR1301 pad 5: (no net) -> Net-(VR1301-Pad5)
Routing:
- net /lpc1549/CANH: track 19.1 -> 30.7 mm
- net /lpc1549/CANL: track 23.0 -> 29.6 mm
Other:
- board text added: "UW HCU 1.3 Usevolt Oy"
- board text removed: "UW HCU 1.2 Usevolt Oy"
